File: wakame_keyboard.kicad_pcb (KiCad board)
At the start: 2 copper layers, 293 x 120 mm, 354 parts, among them J1 USB_C_Receptacle_USB2.0, J2 Conn_02x06_Odd_Even, Q1 BSS138, SW1 SW_Push, U1 Esc, U10 Q, U100 AH49FNTR-G1, U101 AH49FNTR-G1, U102 AH49FNTR-G1, U103 CD74HC4067SM, U104 AH49FNTR-G1, U105 AH49FNTR-G1, U106 AH49FNTR-G1, U107 AH49FNTR-G1, U108 AH49FNTR-G1, U109 AH49FNTR-G1, U11 A, U110 AH49FNTR-G1, U111 AH49FNTR-G1, U112 AH49FNTR-G1, U113 AH49FNTR-G1, U114 CD74HC4067SM, U115 AH49FNTR-G1, U116 AH49FNTR-G1, U117 AH49FNTR-G1, U118 AH49FNTR-G1, U119 AH49FNTR-G1, U12 2, U120 AH49FNTR-G1, U121 AH49FNTR-G1, U122 AH49FNTR-G1, U123 AH49FNTR-G1, U124 CD74HC4067SM, U125 AH49FNTR-G1, U126 AH49FNTR-G1, U127 AH49FNTR-G1, U128 AH49FNTR-G1, U129 AH49FNTR-G1, U13 AH49FNTR-G1, U130 AH49FNTR-G1, U131 AH49FNTR-G1, U132 AH49FNTR-G1, U133 AH49FNTR-G1, U134 AH49FNTR-G1, U135 AH49FNTR-G1, U136 CD74HC4067SM, U137 AH49FNTR-G1, U138 AH49FNTR-G1, U139 AH49FNTR-G1, U14 AH49FNTR-G1, U140 AH49FNTR-G1, U141 AH49FNTR-G1, U142 AH49FNTR-G1, U143 AH49FNTR-G1, U144 AH49FNTR-G1, U145 AH49FNTR-G1, U146 AH49FNTR-G1, U147 CD74HC4067SM, U148 AH49FNTR-G1, U149 AH49FNTR-G1, U15 AH49FNTR-G1, U150 AH49FNTR-G1, U151 AH49FNTR-G1, U152 AH49FNTR-G1, U153 AH49FNTR-G1, U154 AH49FNTR-G1, U155 AH49FNTR-G1, U156 AH49FNTR-G1, U157 AH49FNTR-G1, U158 AH49FNTR-G1, U159 CD74HC4067SM, U16 AH49FNTR-G1, U160 AH49FNTR-G1, U161 AH49FNTR-G1, U162 AH49FNTR-G1, U163 AH49FNTR-G1, U164 AH49FNTR-G1, U165 AH49FNTR-G1, U166 AH49FNTR-G1, U167 AH49FNTR-G1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

Commit message: 配置おおむね完了
Parts:
- R1, R2, SW1: moved to B.Cu
- moved SW1 380.9 mm to (304.0, 110.0), turned to 180 degrees
- moved D82 378.5 mm to (321.5, 208.8)
- moved D81 371.2 mm to (321.7, 189.7)
- moved D77 368.4 mm to (302.4, 208.8)
- moved R85 366.2 mm to (323.9, 207.9), turned to 90 degrees
- moved D76 360.4 mm to (302.8, 189.7)
- moved R84 360.2 mm to (324.1, 188.8), turned to 90 degrees
- moved D78 356.0 mm to (318.3, 152.3), turned to 90 degrees
- moved R80 354.2 mm to (304.8, 207.9), turned to 90 degrees
- moved D71 347.8 mm to (283.4, 208.8)
- moved R79 347.5 mm to (305.2, 188.8), turned to 90 degrees
- moved R81 343.7 mm to (317.3, 149.9), turned to 180 degrees
- moved D73 343.0 mm to (290.5, 168.1)
- moved D80 342.9 mm to (314.3, 130.0)
- moved D64 338.2 mm to (262.0, 206.2)
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