File: wakame_keyboard.kicad_pcb (KiCad board)
At the start: 2 copper layers, 293 x 120 mm, 354 parts, among them J1 USB_C_Receptacle_USB2.0, J2 Conn_02x06_Odd_Even, Q1 BSS138, SW1 SW_Push, U1 Esc, U10 Q, U100 AH49FNTR-G1, U101 AH49FNTR-G1, U102 AH49FNTR-G1, U103 CD74HC4067SM, U104 AH49FNTR-G1, U105 AH49FNTR-G1, U106 AH49FNTR-G1, U107 AH49FNTR-G1, U108 AH49FNTR-G1, U109 AH49FNTR-G1, U11 A, U110 AH49FNTR-G1, U111 AH49FNTR-G1, U112 AH49FNTR-G1, U113 AH49FNTR-G1, U114 CD74HC4067SM, U115 AH49FNTR-G1, U116 AH49FNTR-G1, U117 AH49FNTR-G1, U118 AH49FNTR-G1, U119 AH49FNTR-G1, U12 2, U120 AH49FNTR-G1, U121 AH49FNTR-G1, U122 AH49FNTR-G1, U123 AH49FNTR-G1, U124 CD74HC4067SM, U125 AH49FNTR-G1, U126 AH49FNTR-G1, U127 AH49FNTR-G1, U128 AH49FNTR-G1, U129 AH49FNTR-G1, U13 AH49FNTR-G1, U130 AH49FNTR-G1, U131 AH49FNTR-G1, U132 AH49FNTR-G1, U133 AH49FNTR-G1, U134 AH49FNTR-G1, U135 AH49FNTR-G1, U136 CD74HC4067SM, U137 AH49FNTR-G1, U138 AH49FNTR-G1, U139 AH49FNTR-G1, U14 AH49FNTR-G1, U140 AH49FNTR-G1, U141 AH49FNTR-G1, U142 AH49FNTR-G1, U143 AH49FNTR-G1, U144 AH49FNTR-G1, U145 AH49FNTR-G1, U146 AH49FNTR-G1, U147 CD74HC4067SM, U148 AH49FNTR-G1, U149 AH49FNTR-G1, U15 AH49FNTR-G1, U150 AH49FNTR-G1, U151 AH49FNTR-G1, U152 AH49FNTR-G1, U153 AH49FNTR-G1, U154 AH49FNTR-G1, U155 AH49FNTR-G1, U156 AH49FNTR-G1, U157 AH49FNTR-G1, U158 AH49FNTR-G1, U159 CD74HC4067SM, U16 AH49FNTR-G1, U160 AH49FNTR-G1, U161 AH49FNTR-G1, U162 AH49FNTR-G1, U163 AH49FNTR-G1, U164 AH49FNTR-G1, U165 AH49FNTR-G1, U166 AH49FNTR-G1, U167 AH49FNTR-G1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

Commit message: おおむね完成
Parts:
- added REF**: MountingHole_3.2mm_M3, MountingHole:MountingHole_3.2mm_M3, F.Cu at (41.1, 209.0)
- added REF**: MountingHole_3.2mm_M3, MountingHole:MountingHole_3.2mm_M3, F.Cu at (76.2, 113.3)
- added REF**: MountingHole_3.2mm_M3, MountingHole:MountingHole_3.2mm_M3, F.Cu at (298.9, 149.6)
- added REF**: MountingHole_3.2mm_M3, MountingHole:MountingHole_3.2mm_M3, F.Cu at (272.8, 209.0)
- added REF**: MountingHole_3.2mm_M3, MountingHole:MountingHole_3.2mm_M3, F.Cu at (209.5, 198.5)
- added REF**: MountingHole_3.2mm_M3, MountingHole:MountingHole_3.2mm_M3, F.Cu at (328.1, 170.0)
- added REF**: MountingHole_3.2mm_M3, MountingHole:MountingHole_3.2mm_M3, F.Cu at (41.1, 152.4)
- added REF**: MountingHole_3.2mm_M3, MountingHole:MountingHole_3.2mm_M3, F.Cu at (166.7, 209.0)
- added REF**: MountingHole_3.2mm_M3, MountingHole:MountingHole_3.2mm_M3, F.Cu at (328.1, 95.0)
- added REF**: MountingHole_3.2mm_M3, MountingHole:MountingHole_3.2mm_M3, F.Cu at (62.1, 95.0)
- added REF**: MountingHole_3.2mm_M3, MountingHole:MountingHole_3.2mm_M3, F.Cu at (228.6, 112.8)
- moved Q1 52.5 mm to (45.6, 157.2)
- moved R9 52.5 mm to (48.5, 157.3)
- moved R1 3.41 mm to (188.2, 161.2), turned to -90 degrees
- moved D16 1.78 mm to (95.4, 108.0)
- moved R19 1.78 mm to (97.8, 107.0)
- moved C2 1.72 mm to (294.5, 105.7), turned to 0 degrees
- moved D19 1.52 mm to (114.4, 108.0)
- moved R22 1.52 mm to (116.8, 107.0)
- moved SW1 1.44 mm to (303.0, 111.0)
- moved D1 1.27 mm to (48.1, 108.0)
- moved R3 1.27 mm to (50.5, 107.0)
Routing:
- net +3V3: track 26.0 -> 2462.0 mm, vias 1 -> 12
- net COM_FET: track 0.00 -> 1882.5 mm
- net UART_TX: track 0.00 -> 219.6 mm, vias 0 -> 2
- net RESET: track 0.00 -> 215.2 mm, vias 0 -> 3
- net UART_RX: track 0.00 -> 208.9 mm, vias 0 -> 2
- net SWDIO: track 0.00 -> 158.2 mm
- net SWCLK: track 0.00 -> 149.8 mm
- net LED_PWM: track 0.00 -> 135.4 mm, vias 0 -> 1
- net ADC1_2: track 0.00 -> 113.4 mm
- net +5V: track 27.2 -> 134.4 mm, vias 2 -> 4
- net ADC1_1: track 0.00 -> 66.4 mm
- net ADC2_10: track 0.00 -> 20.4 mm
- net GND: track 24.7 -> 29.3 mm, vias 0 -> 39
- net SELECT_2: track 231.7 -> 229.2 mm, vias 10 -> 6
- net Net-(U79-PB8): track 0.00 -> 1.99 mm
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- added copper zone on B.Cu, net GND
- added copper zone on F.Cu, net GND
Other:
- board text added: "JLCJLCJLCJLC"
